Commit message: task space controller working in simulation

File: kinova_task_space_controller/urdf/gen3.urdf.xacro (robot description, xacro)
@@ -3,5 +3,5 @@
     <!-- Propagate last link name information because it is the gripper's parent link -->
     <xacro:property name="last_arm_link" value="end_effector_link"/>
-    <xacro:macro name="load_arm" params="parent:='' dof vision prefix *origin">
+    <xacro:macro name="load_arm" params="parent:='' simulation:=false dof vision prefix *origin">
         <link name="${prefix}base_link">
             <!-- <inertial>
@@ -62,5 +62,5 @@
         <joint
                 name="${prefix}joint_1"
-                type="continuous">
+                type="revolute">
             <origin xyz="0 0 0.15643" rpy="3.1416 2.7629E-18 -4.9305E-36" />
             <parent
@@ -71,4 +71,6 @@
                     xyz="0 0 1" />
             <limit
+                    lower="-20"
+                    upper="20"
                     effort="39"
                     velocity="1.3963" />
@@ -132,5 +134,5 @@
         <joint
                 name="${prefix}joint_3"
-                type="continuous">
+                type="revolute">
             <origin xyz="0 -0.21038 -0.006375" rpy="-1.5708 1.2326E-32 -2.9122E-16" />
             <parent
@@ -141,4 +143,6 @@
                     xyz="0 0 1" />
             <limit
+                    lower="-20"
+                    upper="20"
                     effort="39"
                     velocity="1.3963" />
@@ -202,5 +206,5 @@
         <joint
                 name="${prefix}joint_5"
-                type="continuous">
+                type="revolute">
             <origin xyz="0 -0.20843 -0.006375" rpy="-1.5708 2.2204E-16 -6.373E-17" />
             <parent
@@ -211,4 +215,6 @@
                     xyz="0 0 1" />
             <limit
+                    lower="-20"
+                    upper="20"
                     effort="9"
                     velocity="1.2218" />
@@ -298,5 +304,5 @@
         <joint
                 name="${prefix}joint_7"
-                type="continuous">
+                type="revolute">
             <origin xyz="0 -0.10593 -0.00017505" rpy="-1.5708 -5.5511E-17 9.6396E-17" />
             <parent
@@ -307,4 +313,6 @@
                     xyz="0 0 1" />
             <limit
+                    lower="-20"
+                    upper="20"
                     effort="9"
                     velocity="1.2218" />
@@ -342,4 +350,14 @@
             </joint>
         </xacro:if>
+        <xacro:if value="${simulation}">
+            <xacro:include filename="$(find kinova_task_space_controller)/urdf/transmission.urdf.xacro" />
+            <xacro:load_gazebo_arm_transmissions prefix="${prefix}"/>
+            <gazebo>
+                <plugin name="gazebo_ros_control" filename="libgazebo_ros_control.so">
+                    <legacyModeNS>true</legacyModeNS>
+                    <!--robotParam>kinova_no_finger</robotParam-->
+                </plugin>
+            </gazebo>
+        </xacro:if>
     </xacro:macro>
 </robot>

File: kinova_task_space_controller/urdf/gen3_standalone.urdf.xacro (robot description, xacro)
@@ -2,5 +2,12 @@
 <robot name="gen3" xmlns:xacro="http://ros.org/wiki/xacro">
     <xacro:include filename="$(find kinova_task_space_controller)/urdf/gen3.urdf.xacro" />
-    <xacro:load_arm parent="" dof="7" vision="false" prefix="">
+    <arg name="simulation" default="false"/>
+    <link name="world"/>
+    <joint name="kinova_base_link" type="fixed">
+        <origin xyz="0 0 0" rpy="0 0 0"/>
+        <parent link="world"/>
+        <child link="arm_base_link"/>
+    </joint>
+    <xacro:load_arm parent="" dof="7" simulation="$(arg simulation)" vision="true" prefix="arm_">
         <origin xyz="0 0 0" rpy="0 0 0"/>
     </xacro:load_arm>
