Commit message: more changes

File: kinova_description_for_controllers/urdf/gen3.urdf.xacro (robot description, xacro)
@@ -71,6 +71,6 @@
                     xyz="0 0 1" />
             <limit
-                    lower="-20"
-                    upper="20"
+                    lower="-6.28"
+                    upper="6.28"
                     effort="39"
                     velocity="1.3963" />
@@ -143,6 +143,6 @@
                     xyz="0 0 1" />
             <limit
-                    lower="-20"
-                    upper="20"
+                    lower="-6.28"
+                    upper="6.28"
                     effort="39"
                     velocity="1.3963" />
@@ -215,6 +215,6 @@
                     xyz="0 0 1" />
             <limit
-                    lower="-20"
-                    upper="20"
+                    lower="-6.28"
+                    upper="6.28"
                     effort="9"
                     velocity="1.2218" />
@@ -313,6 +313,6 @@
                     xyz="0 0 1" />
             <limit
-                    lower="-20"
-                    upper="20"
+                    lower="-6.28"
+                    upper="6.28"
                     effort="9"
                     velocity="1.2218" />
@@ -351,10 +351,9 @@
         </xacro:if>
         <xacro:if value="${simulation}">
-            <xacro:include filename="$(find kinova_task_space_controller)/urdf/transmission.urdf.xacro" />
+            <xacro:include filename="$(find kinova_description_for_controllers)/urdf/transmission.urdf.xacro" />
             <xacro:load_gazebo_arm_transmissions prefix="${prefix}"/>
             <gazebo>
                 <plugin name="gazebo_ros_control" filename="libgazebo_ros_control.so">
                     <legacyModeNS>true</legacyModeNS>
-                    <!--robotParam>kinova_no_finger</robotParam-->
                 </plugin>
             </gazebo>

File: kinova_description_for_controllers/urdf/gen3_standalone.urdf.xacro (robot description, xacro)
@@ -1,13 +1,14 @@
 <?xml version="1.0"?>
 <robot name="gen3" xmlns:xacro="http://ros.org/wiki/xacro">
-    <xacro:include filename="$(find kinova_task_space_controller)/urdf/gen3.urdf.xacro" />
+    <xacro:include filename="$(find kinova_description_for_controllers)/urdf/gen3.urdf.xacro" />
     <arg name="simulation" default="false"/>
+    <arg name="prefix"     default="arm_" />
     <link name="world"/>
     <joint name="kinova_base_link" type="fixed">
         <origin xyz="0 0 0" rpy="0 0 0"/>
         <parent link="world"/>
-        <child link="arm_base_link"/>
+        <child link="$(arg prefix)base_link"/>
     </joint>
-    <xacro:load_arm parent="" dof="7" simulation="$(arg simulation)" vision="true" prefix="arm_">
+    <xacro:load_arm parent="" dof="7" simulation="$(arg simulation)" vision="true" prefix="$(arg prefix)">
         <origin xyz="0 0 0" rpy="0 0 0"/>
     </xacro:load_arm>
