Commit message: adapting simulation to gripper cae

File: kinova_description_for_controllers/urdf/kinova.urdf.xacro (robot description, xacro)
@@ -266,5 +266,5 @@
   <link name="tool_frame"/>
   <joint name="tool_frame_joint" type="fixed">
-    <origin rpy="0 0 0" xyz="0 0 0"/>
+    <origin rpy="0 0 0" xyz="0 0 0.12"/>
     <parent link="end_effector_link"/>
     <child link="tool_frame"/>

File: kinova_missions/kinova_valve_opening/urdf/fake_valve.urdf (robot description, URDF)
Before this commit: robot fake_valve, 3 links, 2 joints
Joints:
- joint valve_base_joint: origin xyz=$(arg x) $(arg y) $(arg z) rpy=3.14 $(arg pitch) $(arg yaw) -> xyz=0.0 0.0 0.5 rpy=3.14 0.0 0.0
