Commit message: working sm with mpc in simulation up to valve rotation

File: kinova_missions/kinova_valve_opening/urdf/fake_valve.urdf.xacro (robot description, xacro)
@@ -50,5 +50,5 @@
       <origin xyz="0 0 0" rpy="0 0 0"/>
       <geometry>
-        <cylinder radius="0.1225" length="0.02"/>
+        <cylinder radius="0.07" length="0.02"/>
       </geometry>
     </visual>
