Commit message: more changes

File: kinova_sensors/zed/zed_descr.urdf.xacro (robot description, xacro)
@@ -22,6 +22,6 @@
     <xacro:property name="baseline" value="0.063" />
     <!-- Arguments -->
-    <xacro:arg name="camera_name"   default="zed" />
-    <xacro:arg name="base_frame"    default="zed_base_link" />
+    <xacro:arg name="camera_name"   default="zedm" />
+    <xacro:arg name="base_frame"    default="zedm_base_link" />
     <xacro:arg name="cam_pos_x"     default="0.11613" />
     <xacro:arg name="cam_pos_y"     default="-0.00775" />
@@ -30,5 +30,5 @@
     <xacro:arg name="cam_pitch"     default="1.570796326" />
     <xacro:arg name="cam_yaw"       default="0.0" />
-       <link name="zed_sensor_mount">
+       <link name="zedm_sensor_mount">
         <visual>
           <origin xyz="0 0 0" rpy="0 0 0" />
@@ -41,5 +41,5 @@
         </visual>
       </link>
-      <joint name="zed_mount_to_zed_link" type="fixed">
+      <joint name="zedm_mount_to_zed_link" type="fixed">
         <origin xyz="0 0 0" rpy="0 0 0"/>
         <parent link="zed_sensor_mount"/>

Commit message: more changes

File: kinova_sensors/zed/zed_descr.urdf.xacro (robot description, xacro)
@@ -43,5 +43,5 @@
       <joint name="zedm_mount_to_zed_link" type="fixed">
         <origin xyz="0 0 0" rpy="0 0 0"/>
-        <parent link="zed_sensor_mount"/>
+        <parent link="zedm_sensor_mount"/>
         <child link="$(arg base_frame)"/>
       </joint>
@@ -58,5 +58,5 @@
             <origin xyz="0 0 0" rpy="0 0 0"/>
             <geometry>
-                <mesh filename="package://zed_wrapper/urdf/models/zedm.stl" />
+                <mesh filename="package://kinova_sensors/zed/models/zedm.stl" />
             </geometry>
             <material name="zedm_mat" />
